File: kicad/murano-keyboard.kicad_pcb (KiCad board)
At the start: 2 copper layers, 23.3 x 63.9 mm, 6 parts, among them P1 CONN_01X04, U1 FEATHER_32U4_BLE

Commit message: Updated to use KiCad 5
Connections:
- R1 pad 1: INPUT_YELLOW -> SIG_YELLOW
- R1 pad 2: SIG_YELLOW -> INPUT_YELLOW
- R2 pad 2: GND -> SIG_GND
- R3 pad 1: INPUT_BLUE -> SIG_BLUE
- R3 pad 2: SIG_BLUE -> INPUT_BLUE
- R4 pad 2: GND -> SIG_GND
- U1 pad 4: GND -> SIG_GND
Routing:
- net SIG_GND: track 0.00 -> 12.7 mm
- net GND: track 12.7 -> 0.00 mm
Changed lines of the file:
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@@
-(kicad_pcb (version 4) (host pcbnew "(2016-02-29 BZR 6601, Git bd80063)-product")
+(kicad_pcb (version 20171130) (host pcbnew 5.0.0)
   (general
-    (links 9)
-    (no_connects 0)
-    (area 137.262799 79.299999 160.755401 143.331001)
     (thickness 1.6)
     (drawings 4)
@@
     (zones 0)
     (modules 6)
-    (nets 31)
+    (nets 32)
   )
   (page A4)
@@
   )
   (setup
-    (last_trace_width 0.762)
+    (last_trace_width 0.25)
     (user_trace_width 0.381)
     (user_trace_width 0.508)
@@
       (layerselection 0x00030_ffffffff)
       (usegerberextensions false)
+      (usegerberattributes false)
+      (usegerberadvancedattributes false)
+      (creategerberjobfile false)
       (excludeedgelayer true)
       (linewidth 0.100000)
@@
       (hpglpennumber 1)
       (hpglpenspeed 20)
-      (hpglpendiameter 15)
+      (hpglpendiameter 15.000000)
       (psnegative false)
       (psa4output false)
@@
   (net 29 "Net-(U1-Pad26)")
   (net 30 "Net-(U1-Pad27)")
+  (net 31 SIG_GND)
   (net_class Default "This is the default net class."
     (clearance 0.2)
@@
     (add_net "Net-(U1-Pad9)")
     (add_net SIG_BLUE)
+    (add_net SIG_GND)
     (add_net SIG_YELLOW)
   )
@@
     (descr "Terminal block 2 pins, Phoenix MSTBA 2,5/4-G-5,08")
     (fp_text reference P1 (at 0 -3.74904) (layer B.SilkS)
-      (effects (font (thickness 0.3048)) (justify mirror))
+      (effects (font (size 1.524 1.524) (thickness 0.3048)) (justify mirror))
     )
     (fp_text value CONN_01X04 (at 0 4.24942) (layer B.SilkS)
-      (effects (font (thickness 0.3048)) (justify mirror))
+      (effects (font (size 1.524 1.524) (thickness 0.3048)) (justify mirror))
     )
     (fp_line (start 11.1506 9.99998) (end -11.1506 9.99998) (layer B.SilkS) (width 0.254))
@@
     (fp_line (start 11.25 1.6) (end -1.05 1.6) (layer B.CrtYd) (width 0.05))
     (pad 1 thru_hole circle (at 0 0 270) (size 2.2 2.2) (drill 0.8) (layers *.Cu *.Mask)
+      (net 2 SIG_YELLOW))
+    (pad 2 thru_hole oval (at 10.16 0 270) (size 2.2 2.2) (drill 0.8) (layers *.Cu *.Mask)
       (net 5 INPUT_YELLOW))
-    (pad 2 thru_hole oval (at 10.16 0 270) (size 2.2 2.2) (drill 0.8) (layers *.Cu *.Mask)
-      (net 2 SIG_YELLOW))
     (model Resistors_THT.3dshapes/R_Axial_DIN0207_L6.3mm_D2.5mm_P10.16mm_Horizontal.wrl
       (at (xyz 0 0 0))
@@
       (net 5 INPUT_YELLOW))
     (pad 2 thru_hole oval (at 10.16 0 90) (size 2.2 2.2) (drill 0.8) (layers *.Cu *.Mask)
-      (net 3 GND))
+      (net 31 SIG_GND))
     (model Resistors_THT.3dshapes/R_Axial_DIN0207_L6.3mm_D2.5mm_P10.16mm_Horizontal.wrl
       (at (xyz 0 0 0))
@@
     (fp_line (start 11.25 1.6) (end -1.05 1.6) (layer B.CrtYd) (width 0.05))
     (pad 1 thru_hole circle (at 0 0 270) (size 2.2 2.2) (drill 0.8) (layers *.Cu *.Mask)
+      (net 4 SIG_BLUE))
+    (pad 2 thru_hole oval (at 10.16 0 270) (size 2.2 2.2) (drill 0.8) (layers *.Cu *.Mask)
       (net 6 INPUT_BLUE))
-    (pad 2 thru_hole oval (at 10.16 0 270) (size 2.2 2.2) (drill 0.8) (layers *.Cu *.Mask)
-      (net 4 SIG_BLUE))
     (model Resistors_THT.3dshapes/R_Axial_DIN0207_L6.3mm_D2.5mm_P10.16mm_Horizontal.wrl
       (at (xyz 0 0 0))
@@
       (net 6 INPUT_BLUE))
     (pad 2 thru_hole oval (at 10.16 0 90) (size 2.2 2.2) (drill 0.8) (layers *.Cu *.Mask)
-      (net 3 GND))
+      (net 31 SIG_GND))
     (model Resistors_THT.3dshapes/R_Axial_DIN0207_L6.3mm_D2.5mm_P10.16mm_Horizontal.wrl
       (at (xyz 0 0 0))
@@
       (net 8 "Net-(U1-Pad3)"))
     (pad 4 thru_hole circle (at -10.16 11.43 180) (size 2.2 2.2) (drill 0.8) (layers *.Cu *.Mask B.SilkS)
-      (net 3 GND))
+      (net 31 SIG_GND))
     (pad 5 thru_hole circle (at -10.16 8.89 180) (size 2.2 2.2) (drill 0.8) (layers *.Cu *.Mask B.SilkS)
       (net 9 "Net-(U1-Pad5)"))
@@
   (gr_line (start 137.3378 79.375) (end 160.6804 79.375) (angle 90) (layer Edge.Cuts) (width 0.15))
   (segment (start 146.46 133) (end 146.46 120.16) (width 0.762) (layer F.Cu) (net 2) (status C00000))
-  (segment (start 151.54 93.57) (end 159.16 93.57) (width 0.762) (layer F.Cu) (net 3) (status C00000))
-  (segment (start 146.46 93.57) (end 151.54 93.57) (width 0.762) (layer F.Cu) (net 3))
+  (segment (start 151.54 93.57) (end 159.16 93.57) (width 0.762) (layer F.Cu) (net 31) (status C00000))
+  (segment (start 146.46 93.57) (end 151.54 93.57) (width 0.762) (layer F.Cu) (net 31))
   (segment (start 151.54 133) (end 151.54 120.16) (width 0.762) (layer F.Cu) (net 4) (status C00000))
   (segment (start 146.46 110) (end 146.46 103.73) (width 0.762) (layer F.Cu) (net 5) (status C00000))
